File: raptor/raptor/raptor.sch (KiCad schematic (older format))
At the start: 7 parts, among them P1 Digital, P2 CONN_01X02, P3 CONN_02X08, P4 Analog, P5 CONN_01X08, P6 CONN_01X08, P7 CONN_01X02

Commit message: Add files via upload
Parts:
- added BT? (x2): Battery_Cell, symbol Battery_Cell
Connections:
- net 4: now also P3.8 (P8); no longer P3.2 (P2)
- net 6(**): now also P3.6 (P6); no longer P3.4 (P4)
- net 8: now also P1.11 (P11), P3.4 (P4); no longer P3.6 (P6)
- net 9(**): now also P3.2 (P2); no longer P3.8 (P8)
- net A0: now also P3.16 (P16); no longer P3.10 (P10)
- net A1: now also P3.14 (P14); no longer P3.12 (P12)
- net A2: now also P3.12 (P12); no longer P3.14 (P14)
- net A3: now also P3.10 (P10); no longer P3.16 (P16)
- net GND: now also P1.3 (P3), BT?.2 (-)
- net Reset: no longer P1.3 (P3)
- new net: BT?.1 (+), BT?.2 (-)
- no-connect marks 12 -> 10
Other:
- note added: "Chasis PCB para Robot Raptor siguelíneas con motores N20 y sensor Pololu QTR-8x"
- note added: "Pololu QTR 8x sensor"
- note added: "TB6612FNG driver"
- moved on the sheet: P1, P2, P4, P5, P6, P7

Commit message: Add files via upload
Parts:
- added R?: R, symbol R
- added SW?: SW_SPST, symbol SW_SPST
- added SW?: SW_PUSHBUTTON, symbol SW_PUSHBUTTON
Connections:
- net 7: now also R?.1, SW?.1
- net GND: now also R?.2
- net RAW: now also SW?.1
- net VCC: now also SW?.2
- net at BT?.1 (+): now also SW?.2
- no-connect marks 10 -> 9
Other:
- note added: "2 x 16340 batteries"
- moved on the sheet: BT?
Changed lines of the file:
@@
 NoConn ~ 3950 1700
 NoConn ~ 4150 1700
-NoConn ~ 3000 4200
 Text Notes 7050 6700 0    60   ~ 0
 Chasis PCB para Robot Raptor siguelíneas con motores N20 y sensor Pololu QTR-8x
@@
 	2200 4100 3350 4100
 Wire Wire Line
-	3000 4200 3350 4200
+	1450 4200 3350 4200
 Wire Wire Line
 	2000 4400 3350 4400
@@
 Connection ~ 4350 2850
 Wire Wire Line
-	7300 2850 6750 2850
-Wire Wire Line
-	7300 2850 7300 3150
+	8050 2850 7500 2850
 $Comp
 L Battery_Cell BT?
 U 1 1 5894BE1A
-P 7300 3350
-F 0 "BT?" H 7400 3450 50  0000 L CNN
-F 1 "Battery_Cell" H 7400 3350 50  0000 L CNN
-F 2 "" V 7300 3410 50  0000 C CNN
-F 3 "" V 7300 3410 50  0000 C CNN
-	1    7300 3350
+P 8050 3800
+F 0 "BT?" H 8150 3900 50  0000 L CNN
+F 1 "Battery_Cell" H 8150 3800 50  0000 L CNN
+F 2 "" V 8050 3860 50  0000 C CNN
+F 3 "" V 8050 3860 50  0000 C CNN
+	1    8050 3800
 	1    0    0    -1
 $EndComp
@@
 L Battery_Cell BT?
 U 1 1 5894BE6F
-P 7300 3850
-F 0 "BT?" H 7400 3950 50  0000 L CNN
-F 1 "Battery_Cell" H 7400 3850 50  0000 L CNN
-F 2 "" V 7300 3910 50  0000 C CNN
-F 3 "" V 7300 3910 50  0000 C CNN
-	1    7300 3850
-	1    0    0    -1
-$EndComp
-Wire Wire Line
-	7300 3450 7300 3650
-Wire Wire Line
-	7300 3950 7300 4150
+P 8050 4300
+F 0 "BT?" H 8150 4400 50  0000 L CNN
+F 1 "Battery_Cell" H 8150 4300 50  0000 L CNN
+F 2 "" V 8050 4360 50  0000 C CNN
+F 3 "" V 8050 4360 50  0000 C CNN
+	1    8050 4300
+	1    0    0    -1
+$EndComp
+Wire Wire Line
+	8050 3900 8050 4100
+Wire Wire Line
+	8050 4400 8050 4850
 $Comp
 L GND #PWR?
 U 1 1 5894BFC1
-P 7300 4150
-F 0 "#PWR?" H 7300 3900 50  0001 C CNN
-F 1 "GND" H 7300 4000 50  0000 C CNN
-F 2 "" H 7300 4150 50  0000 C CNN
-F 3 "" H 7300 4150 50  0000 C CNN
-	1    7300 4150
+P 8050 4850
+F 0 "#PWR?" H 8050 4600 50  0001 C CNN
+F 1 "GND" H 8050 4700 50  0000 C CNN
+F 2 "" H 8050 4850 50  0000 C CNN
+F 3 "" H 8050 4850 50  0000 C CNN
+	1    8050 4850
 	1    0    0    -1
 $EndComp
@@
 Wire Wire Line
 	3350 3500 3250 3500
+$Comp
+L SW_SPST SW?
+U 1 1 5894A3B3
+P 7000 2850
+F 0 "SW?" H 6900 2950 70  0000 C CNN
+F 1 "SW_SPST" H 7000 2750 70  0000 C CNN
+F 2 "" H 7000 2850 60  0000 C CNN
+F 3 "" H 7000 2850 60  0000 C CNN
+	1    7000 2850
+	1    0    0    -1
+$EndComp
+Wire Notes Line
+	7600 4700 8800 4700
+Wire Notes Line
+	8800 4700 8800 3200
+Wire Notes Line
+	8800 3200 7600 3200
+Wire Notes Line
+	7600 3200 7600 4700
+Text Notes 7700 3350 0    60   ~ 0
+2 x 16340 batteries
+$Comp
+L VCC #PWR?
+U 1 1 5894A764
+P 1450 3600
+F 0 "#PWR?" H 1450 3450 50  0001 C CNN
+F 1 "VCC" H 1450 3750 50  0000 C CNN
+F 2 "" H 1450 3600 50  0000 C CNN
+F 3 "" H 1450 3600 50  0000 C CNN
+	1    1450 3600
+	1    0    0    -1
+$EndComp
+$Comp
+L SW_PUSHBUTTON SW?
+U 1 1 5894A78C
+P 1450 3900
+F 0 "SW?" H 1300 4010 50  0000 C CNN
+F 1 "SW_PUSHBUTTON" H 1450 3820 50  0000 C CNN
+F 2 "" H 1450 3900 60  0000 C CNN
+F 3 "" H 1450 3900 60  0000 C CNN
+	1    1450 3900
+	0    -1   -1   0
+$EndComp
+$Comp
+L R R?
+U 1 1 5894A80B
+P 1450 4450
+F 0 "R?" V 1530 4450 50  0000 C CNN
+F 1 "R" V 1450 4450 50  0000 C CNN
+F 2 "" H 1450 4450 60  0000 C CNN
+F 3 "" H 1450 4450 60  0000 C CNN
+	1    1450 4450
+	1    0    0    -1
+$EndComp
+$Comp
+L GND #PWR?
+U 1 1 5894A880
+P 1450 4700
+F 0 "#PWR?" H 1450 4450 50  0001 C CNN
+F 1 "GND" H 1450 4550 50  0000 C CNN
+F 2 "" H 1450 4700 50  0000 C CNN
+F 3 "" H 1450 4700 50  0000 C CNN
+	1    1450 4700
+	1    0    0    -1
+$EndComp
+Connection ~ 1450 4200
+Wire Wire Line
+	8050 2850 8050 3600
 $EndSCHEMATC

Commit message: Add files via upload
Parts:
- removed P2, P7: CONN_01X02, symbol CONN_01X02
- removed SW?: SW_SPST, symbol SW_SPST
- added P10: CONN_01X05, symbol CONN_01X05
- added P2, P7, P8, P9: CONN_01X01, symbol CONN_01X01
- gave numbers to parts that had none: 4
Connections:
- net RAW: now also P10.3 (P3)
- net at P6.7 (P7): now also P8.1 (P1)
- net at P6.6 (P6): now also P9.1 (P1)
- net at P6.5 (P5): now also P7.1 (P1)
- net at P6.4 (P4): now also P2.1 (P1)
- net at BT16340_1.1 (+): now also P10.4 (P4)
- no-connect marks 9 -> 12
